File: Palac.kicad_sch (KiCad schematic)
At the start: 70 parts, among them J2 4PIN, SW1 SW_PUSH, SW10 SW_PUSH, SW11 SW_PUSH, SW12 SW_PUSH, SW13 SW_PUSH, SW14 SW_PUSH, SW15 SW_PUSH, SW16 SW_PUSH, SW17 SW_PUSH, SW18 SW_PUSH, SW19 SW_PUSH, SW2 SW_PUSH, SW20 SW_PUSH, SW21 SW_PUSH, SW22 SW_PUSH, SW23 SW_PUSH, SW24 SW_PUSH, SW25 SW_PUSH, SW26 SW_PUSH, SW27 SW_PUSH, SW28 SW_PUSH, SW29 SW_PUSH, SW3 SW_PUSH, SW30 SW_PUSH, SW4 SW_PUSH, SW5 SW_PUSH, SW6 SW_PUSH, SW7 SW_PUSH, SW8 SW_PUSH, SW9 SW_PUSH, U1 ProMicro

Commit message: Updated layout
Parts:
- added SW99: SW_PUSH, Palac:CherryMX_Hotswap, symbol Palac:SW_PUSH-Lily58-cache-Lily58_Pro-rescue
- D1, D10, D11, D12, D13, D14, D15, D16, D17, D18, D19, D2, D20, D21, D22, D23, D24, D25, D26, D27, D28, D29, D3, D30, D4, D5, D6, D7, D8, D9: footprint SofleKeyboard-footprint:Diode_SOD123 -> Palac:Diode_SOD123; symbol SofleKeyboard-rescue:D-Lily58-cache-Lily58_Pro-rescue -> Palac:D-Lily58-cache-Lily58_Pro-rescue
- J2: footprint SofleKeyboard-footprint:MJ-4PP-9 -> Palac:MJ-4PP-9; symbol SofleKeyboard-rescue:MJ-4PP-9-Lily58-cache-Lily58_Pro-rescue -> Palac:MJ-4PP-9-Lily58-cache-Lily58_Pro-rescue
- R1, R2: footprint SofleKeyboard-footprint:R_1206_DoubleSided -> Palac:R_1206_DoubleSided; symbol SofleKeyboard-rescue:R-Lily58-cache-Lily58_Pro-rescue -> Palac:R-Lily58-cache-Lily58_Pro-rescue
- RSW1: footprint SofleKeyboard-footprint:TACT_SWITCH_TVBP06 -> Palac:TACT_SWITCH_TVBP06; symbol SofleKeyboard-rescue:SW_RST-Lily58-cache-Lily58_Pro-rescue -> Palac:SW_RST-Lily58-cache-Lily58_Pro-rescue
- SW1, SW10, SW11, SW12, SW13, SW14, SW15, SW16, SW17, SW18, SW19, SW2, SW20, SW21, SW22, SW23, SW24, SW25, SW26, SW27, SW28, SW29, SW3, SW30, SW4, SW5, SW6, SW7, SW8, SW9: footprint SofleKeyboard-footprint:CherryMX_Hotswap -> Palac:CherryMX_Hotswap; symbol SofleKeyboard-rescue:SW_PUSH-Lily58-cache-Lily58_Pro-rescue -> Palac:SW_PUSH-Lily58-cache-Lily58_Pro-rescue
- TH3, TH4, TH5, TH6, TH7: footprint SofleKeyboard-footprint:HOLE_M2_TH -> Palac:HOLE_M2_TH; symbol SofleKeyboard-rescue:HOLE-Lily58-cache-Lily58_Pro-rescue -> Palac:HOLE-Lily58-cache-Lily58_Pro-rescue
- U1: footprint SofleKeyboard-footprint:ArduinoProMicro-ZigZag-DoubleSided -> Palac:ArduinoProMicro-ZigZag-DoubleSided; symbol SofleKeyboard-rescue:ProMicro_2-Lily58-cache-Lily58_Pro-rescue -> Palac:ProMicro_2-Lily58-cache-Lily58_Pro-rescue
Connections:
- net colT: now reaches U1.19 (A2(PF5))
- net colT: now also SW99.2
- net rowT: now reaches U1.7 (D4(PD4))
- net rowT: now also SW99.1
- no-connect marks 6 -> 4
Other:
- moved on the sheet: D1, D10, D11, D12, D13, D14, D15, D16, D17, D18, D19, D2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

Commit message: Tidy
Connections:
- net GND: now also SW99.1
- net colT renamed SW99
- net rowT: no longer names the net of U1.7 (D4(PD4))
- net rowT: no longer SW99.1
- no-connect marks 4 -> 5
Changed lines of the file:
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@@
   (junction (at 185.42 81.28) (diameter 0) (color 0 0 0 0)
-  )
-  (junction (at 35.56 60.96) (diameter 0) (color 0 0 0 0)
   )
   (junction (at 185.42 64.77) (diameter 0) (color 0 0 0 0)
@@
   (no_connect (at 68.58 63.5))
   (no_connect (at 68.58 53.34))
+  (no_connect (at 35.56 68.58))
   (no_connect (at 35.56 53.34))
   (wire (pts (xy 149.86 106.68) (xy 149.86 123.19))
@@
     (stroke (width 0) (type default))
   )
-  (wire (pts (xy 26.67 60.96) (xy 35.56 60.96))
-    (stroke (width 0) (type default))
-  )
   (wire (pts (xy 165.1 97.79) (xy 143.51 97.79))
     (stroke (width 0) (type default))
@@
     )
   )
-  (global_label "colT" (shape input) (at 68.58 66.04 0) (fields_autoplaced)
-    (effects (font (size 1.27 1.27)) (justify left))
-    (property "Intersheetrefs" "${INTERSHEET_REFS}" (at 74.702 66.04 0)
+  (global_label "SW99" (shape input) (at 68.58 66.04 0) (fields_autoplaced)
+    (effects (font (size 1.27 1.27)) (justify left))
+    (property "Intersheetrefs" "${INTERSHEET_REFS}" (at 75.9115 66.04 0)
       (effects (font (size 1.27 1.27)) (justify left) hide)
     )
@@
     )
   )
-  (global_label "GND" (shape input) (at 26.67 60.96 180) (fields_autoplaced)
-    (effects (font (size 1.27 1.27)) (justify right))
-    (property "Intersheetrefs" "${INTERSHEET_REFS}" (at 20.5479 60.96 0)
-      (effects (font (size 1.27 1.27)) (justify right) hide)
-    )
-  )
-  (global_label "colT" (shape input) (at 115.57 82.55 0) (fields_autoplaced)
-    (effects (font (size 1.27 1.27)) (justify left))
-    (property "Intersheetrefs" "${INTERSHEET_REFS}" (at 121.692 82.55 0)
-      (effects (font (size 1.27 1.27)) (justify left) hide)
-    )
-  )
-  (global_label "rowT" (shape input) (at 35.56 68.58 180) (fields_autoplaced)
-    (effects (font (size 1.27 1.27)) (justify right))
-    (property "Intersheetrefs" "${INTERSHEET_REFS}" (at 29.0751 68.58 0)
-      (effects (font (size 1.27 1.27)) (justify right) hide)
+  (global_label "GND" (shape input) (at 35.56 60.96 180) (fields_autoplaced)
+    (effects (font (size 1.27 1.27)) (justify right))
+    (property "Intersheetrefs" "${INTERSHEET_REFS}" (at 29.4379 60.96 0)
+      (effects (font (size 1.27 1.27)) (justify right) hide)
+    )
+  )
+  (global_label "SW99" (shape input) (at 115.57 82.55 0) (fields_autoplaced)
+    (effects (font (size 1.27 1.27)) (justify left))
+    (property "Intersheetrefs" "${INTERSHEET_REFS}" (at 122.9015 82.55 0)
+      (effects (font (size 1.27 1.27)) (justify left) hide)
     )
   )
@@
     )
   )
-  (global_label "rowT" (shape input) (at 100.33 82.55 180) (fields_autoplaced)
-    (effects (font (size 1.27 1.27)) (justify right))
-    (property "Intersheetrefs" "${INTERSHEET_REFS}" (at 93.8451 82.55 0)
-      (effects (font (size 1.27 1.27)) (justify right) hide)
-    )
+  (global_label "GND" (shape input) (at 100.33 82.55 180) (fields_autoplaced)
+    (effects (font (size 1.27 1.27)) (justify right))
+    (property "Intersheetrefs" "${INTERSHEET_REFS}" (at 94.2079 82.55 0)
+      (effects (font (size 1.27 1.27)) (justify right) hide)
+    )
